Commit message: Fixing the tricycle urdf file

File: install/description/share/description/urdf/tricycle.urdf (robot description, URDF)
Before this commit: robot tricycle, 4 links, 3 joints
Links:
- removed link bwheel
- removed link lwheel
- removed link rwheel
- added link bwheel_left, mass 0.12; collision cylinder length=0.04 radius=0.05; visual cylinder length=0.04 radius=0.05
- added link bwheel_right, mass 0.12; collision cylinder length=0.04 radius=0.05; visual cylinder length=0.04 radius=0.05
- added link fork, mass 0.2; collision box size=0.05 0.05 0.1; visual box size=0.05 0.05 0.1
- added link fwheel, mass 0.12; collision cylinder length=0.04 radius=0.05; visual cylinder length=0.04 radius=0.05
Joints:
- removed joint base_to_bwheel
- removed joint base_to_lwheel
- added joint base_to_bwheel_left: type continuous, parent base_link, child bwheel_left, origin xyz=-0.17 0.17 -0.1 rpy=-1.5708 0 0, axis 0 0 1
- added joint fork_to_fwheel: type continuous, parent fork, child fwheel, origin xyz=0 0 -0.1 rpy=-1.5708 0 0, axis 0 0 1
- added joint steer_joint: type revolute, parent base_link, child fork, origin xyz=0.15 0 0.0 rpy=0 0 0, axis 0 0 1, limit lower=-0.6 upper=0.6 effort=10 velocity=2.0
- joint base_to_rwheel: child rwheel -> bwheel_right; origin xyz=0.15 -0.15 -0.1 rpy=-1.5708 0 0 -> xyz=-0.17 -0.17 -0.1 rpy=-1.5708 0 0

File: src/description/urdf/tricycle.urdf (robot description, URDF)
Before this commit: robot tricycle, 4 links, 3 joints
Links:
- removed link bwheel
- removed link lwheel
- removed link rwheel
- added link bwheel_left, mass 0.12; collision cylinder length=0.04 radius=0.05; visual cylinder length=0.04 radius=0.05
- added link bwheel_right, mass 0.12; collision cylinder length=0.04 radius=0.05; visual cylinder length=0.04 radius=0.05
- added link fork, mass 0.2; collision box size=0.05 0.05 0.1; visual box size=0.05 0.05 0.1
- added link fwheel, mass 0.12; collision cylinder length=0.04 radius=0.05; visual cylinder length=0.04 radius=0.05
Joints:
- removed joint base_to_bwheel
- removed joint base_to_lwheel
- added joint base_to_bwheel_left: type continuous, parent base_link, child bwheel_left, origin xyz=-0.17 0.17 -0.1 rpy=-1.5708 0 0, axis 0 0 1
- added joint fork_to_fwheel: type continuous, parent fork, child fwheel, origin xyz=0 0 -0.1 rpy=-1.5708 0 0, axis 0 0 1
- added joint steer_joint: type revolute, parent base_link, child fork, origin xyz=0.15 0 0.0 rpy=0 0 0, axis 0 0 1, limit lower=-0.6 upper=0.6 effort=10 velocity=2.0
- joint base_to_rwheel: child rwheel -> bwheel_right; origin xyz=0.15 -0.15 -0.1 rpy=-1.5708 0 0 -> xyz=-0.17 -0.17 -0.1 rpy=-1.5708 0 0

Commit message: Added camera

File: install/description/share/description/urdf/tricycle.urdf (robot description, URDF)
Before this commit: robot tricycle, 5 links, 4 joints
Links:
- added link camera_link; visual box size=0.05 0.05 0.05
Joints:
- added joint base_to_camera: type fixed, parent base_link, child camera_link, origin xyz=0 0 0 rpy=0 0 0

Commit message: Fixed camera positioning and front wheel

File: install/description/share/description/urdf/tricycle.urdf (robot description, URDF)
Before this commit: robot tricycle, 6 links, 5 joints
Joints:
- joint base_to_camera: origin xyz=0 0 0 rpy=0 0 0 -> xyz=0.15 0 0.12 rpy=0 0 0
- joint fork_to_fwheel: origin xyz=0 0 -0.1 rpy=-1.5708 0 0 -> xyz=0 0 -0.12 rpy=-1.5708 0 0

Commit message: Camera Fix

File: install/description/share/description/urdf/tricycle.urdf (robot description, URDF)
Before this commit: robot tricycle, 6 links, 5 joints
Joints:
- joint steer_joint: axis 0 0 1 -> 0 1 0

Commit message: .

File: install/description/share/description/urdf/tricycle.urdf (robot description, URDF)
Before this commit: robot tricycle, 6 links, 5 joints
Joints:
- joint fork_to_fwheel: origin xyz=0 0 -0.12 rpy=-1.5708 0 0 -> xyz=0 0 -0.14 rpy=-1.5708 0 0
- joint steer_joint: axis 0 1 0 -> 0 0 1

Commit message: Fixed the camera and made it stop when too close

File: install/description/share/description/urdf/tricycle.urdf (robot description, URDF)
Before this commit: robot tricycle, 6 links, 5 joints
Links:
- link camera_link: mass None -> 0.05
Joints:
- joint base_to_bwheel_left: origin xyz=-0.17 0.17 -0.1 rpy=-1.5708 0 0 -> xyz=-0.17 0.17 -0.14 rpy=-1.5707 0 0
- joint base_to_camera: origin xyz=0.15 0 0.12 rpy=0 0 0 -> xyz=0.2 0 0.20 rpy=0 0 0
- joint base_to_rwheel: origin xyz=-0.17 -0.17 -0.1 rpy=-1.5708 0 0 -> xyz=-0.17 -0.17 -0.14 rpy=-1.5707 0 0
- joint fork_to_fwheel: origin xyz=0 0 -0.14 rpy=-1.5708 0 0 -> xyz=0 0 -0.14 rpy=-1.5707 0 0

Commit message: fixed camera positioning

File: install/description/share/description/urdf/tricycle.urdf (robot description, URDF)
Before this commit: robot tricycle, 6 links, 5 joints
Joints:
- joint base_to_camera: origin xyz=0.2 0 0.20 rpy=0 0 0 -> xyz=0.2 0 0.12 rpy=0 0 0
